File: Hardware/RemoteDTMF/RemoteDTMF.kicad_pcb (KiCad board)
At the start: 2 copper layers, 88.9 x 59.7 mm, 35 parts, among them J1 REG. 7V, J10 MT8870D, J2 BATT 12V, J3 P12V, J4 Analog, J5 Digital, J6 TRX TELCO, J7 AL. ATTINY85, J8 IO ATTINY85, J9 AT-D578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

Commit message: Update Schematic & WIP 0.6A
Parts:
- added D1: LED, LED_THT:LED_D3.0mm, F.Cu at (149.5, 143.2)
- added D2: LED, LED_THT:LED_D3.0mm, F.Cu at (149.5, 161.0)
- added J11: P12V2, Connector_PinHeader_2.54mm:PinHeader_1x01_P2.54mm_Vertical, F.Cu at (198.3, 118.6)
- added J12: RELAY 1, TerminalBlock:TerminalBlock_MaiXu_MX126-5.0-02P_1x02_P5.00mm, F.Cu at (150.8, 136.8)
- added J13: RELAY 2, TerminalBlock:TerminalBlock_MaiXu_MX126-5.0-02P_1x02_P5.00mm, F.Cu at (150.8, 154.6)
- added J14: P0, Connector_PinHeader_2.54mm:PinHeader_1x10_P2.54mm_Vertical, F.Cu at (72.0, 145.7)
- added J15: P1, Connector_PinHeader_2.54mm:PinHeader_1x10_P2.54mm_Vertical, F.Cu at (92.4, 145.7)
- added J16: PCF8575, Connector_PinHeader_2.54mm:PinHeader_1x05_P2.54mm_Vertical, F.Cu at (87.3, 140.6)
- added J17: DS3231, Connector_PinHeader_2.54mm:PinHeader_1x06_P2.54mm_Vertical, F.Cu at (205.5, 78.9)
- added J18: BME280, Connector_PinHeader_2.54mm:PinHeader_1x04_P2.54mm_Vertical, F.Cu at (198.3, 106.3)
- added J19: BME280, Connector_PinHeader_2.54mm:PinHeader_1x04_P2.54mm_Vertical, F.Cu at (202.9, 106.3)
- added R10: 4K7, Resistor_THT:R_Axial_DIN0204_L3.6mm_D1.6mm_P7.62mm_Horizontal, F.Cu at (135.6, 144.4)
- added R11: 4K7, Resistor_THT:R_Axial_DIN0204_L3.6mm_D1.6mm_P7.62mm_Horizontal, F.Cu at (135.5, 161.1)
- added R12: 470R, Resistor_THT:R_Axial_DIN0204_L3.6mm_D1.6mm_P7.62mm_Horizontal, F.Cu at (194.1, 90.8)
- added R13: 470R, Resistor_THT:R_Axial_DIN0204_L3.6mm_D1.6mm_P7.62mm_Horizontal, F.Cu at (194.1, 93.9)
- added R8: 2K2, Resistor_THT:R_Axial_DIN0204_L3.6mm_D1.6mm_P7.62mm_Horizontal, F.Cu at (194.1, 78.2)
- added R9: 100K, Resistor_THT:R_Axial_DIN0204_L3.6mm_D1.6mm_P7.62mm_Horizontal, F.Cu at (194.1, 81.3)
- added RLY1: G5QU-1A, Relay_THT:Relay_SPST_Omron-G5Q-1A, F.Cu at (125.4, 139.4)
- added RLY2: G5QU-1A, Relay_THT:Relay_SPST_Omron-G5Q-1A, F.Cu at (125.4, 157.2)
- added U4: PC817, Package_DIP:DIP-4_W7.62mm, F.Cu at (173.1, 120.2)
- added U5: ULN2803A, Package_DIP:DIP-18_W7.62mm, F.Cu at (110.1, 134.3)
- added U6: P82B715D, Package_DIP:DIP-8_W7.62mm, F.Cu at (185.0, 116.2)
- J3: value P12V -> P12V1
Connections:
- net /CMDPTT renamed /CMD_PTT
- net Net-(J3-Pin_1) renamed /P12V1
- J4 pad 8: /A4/SDA -> /SDA
- J4 pad 9: /A5/SCL -> /SCL
- J5 pad 10: /PRES12V -> /~{STQ}
- J5 pad 11: /~{STQ} -> /~{INT}
- R3 pad 2: /PRES12V -> /PRES12V1
- U1 pad 4: /PRES12V -> /PRES12V1
- U3 pad 12: unconnected-(U3-Pad12) -> GND
- U3 pad 6: unconnected-(U3-Pad6) -> GND
Routing:
- net /PRES12V: track 23.1 -> 0.00 mm
- net /~{STQ}: track 23.0 -> 46.1 mm
- removed copper zone on B.Cu, net GND
- removed copper zone on F.Cu, net GND
Other:
- board text added: "REMOTE DTMF AT-D578 NICOLAS F4ISE - V1B"
- board text removed: "REMOTE DTMF AT-D578 NICOLAS F4ISE - V1A"

Commit message: WIP Update PCB 2
Parts:
- removed J11: P12V2, Connector_PinHeader_2.54mm:PinHeader_1x01_P2.54mm_Vertical
- removed J3: P12V1, Connector_PinHeader_2.54mm:PinHeader_1x01_P2.54mm_Vertical
- moved J17 112.2 mm to (93.7, 88.6), turned to -90 degrees
- moved R9 84.2 mm to (121.5, 124.1), turned to -90 degrees
- moved J9 75.0 mm to (152.1, 70.0), turned to 90 degrees
- moved R8 73.9 mm to (143.1, 131.7), turned to 180 degrees
- moved J18 60.4 mm to (140.6, 88.5), turned to 180 degrees
- moved J19 50.3 mm to (155.9, 88.5), turned to 180 degrees
- moved U6 50.2 mm to (152.0, 78.4), turned to -90 degrees
- moved J14 46.2 mm to (78.3, 99.9)
- moved J15 46.2 mm to (98.6, 99.9)
- moved J16 46.2 mm to (93.5, 94.8)
- moved U4 43.0 mm to (131.7, 131.7), turned to 180 degrees
- moved R12 34.5 mm to (159.7, 88.5), turned to 90 degrees
- moved RLY2 32.2 mm to (135.5, 126.6)
- moved RLY1 32.2 mm to (135.5, 108.8)
- moved R10 32.2 mm to (145.6, 113.9)
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Connections:
- net Net-(J12-Pin_2) renamed /P12V1S
- net Net-(J13-Pin_2) renamed /P12V2S
- J19 pad 3: /SCLX -> /LCL
- J19 pad 4: /SDAX -> /LDA
- R12 pad 2: /SCLX -> /LDA
- R13 pad 2: /SDAX -> /LCL
- U6 pad 2: /SCLX -> /LDA
- U6 pad 3: /SCL -> /SDA
- U6 pad 6: /SDA -> /SCL
- U6 pad 7: /SDAX -> /LCL
Routing:
- net +5V: track 185.5 -> 349.6 mm, vias 2 -> 1
- net /SCL: track 0.00 -> 95.6 mm
- net /SDA: track 0.00 -> 93.1 mm
- net /~{INT}: track 0.00 -> 85.9 mm, vias 0 -> 4
- net /MIC: track 86.3 -> 2.54 mm, vias 1 -> 0
- net /URX: track 78.2 -> 0.00 mm
- net /UTX: track 76.9 -> 0.00 mm
- net /DTMF: track 67.6 -> 0.00 mm, vias 1 -> 0
- net /CMD_PTT: track 48.4 -> 92.5 mm, vias 0 -> 2
- net /PRES12V2: track 0.00 -> 42.4 mm, vias 0 -> 1
- net /CW: track 45.1 -> 3.81 mm, vias 1 -> 0
- net /CMD_RLY21: track 0.00 -> 33.5 mm
- net VCC: track 34.9 -> 68.1 mm
- net /PRES12V1: track 0.00 -> 32.9 mm
- net /CMD_RLY25: track 0.00 -> 30.3 mm
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- added copper zone on B.Cu, net /P12V1
- added copper zone on F.Cu, net /P12V1
- added copper zone on B.Cu, net /P12V1S
- added copper zone on F.Cu, net /P12V1S
- added copper zone on B.Cu, net /P12V2
- added copper zone on F.Cu, net /P12V2
- added copper zone on B.Cu, net /P12V2S
- added copper zone on F.Cu, net /P12V2S
- added copper zone on B.Cu, net GND
- added copper zone on F.Cu, net GND
Other:
- board size 88.9 x 59.7 mm -> 100.3 x 104.1 mm
- board text removed: "ICSP"
- board text removed: "USB Mini-B"

Commit message: WIP Update PCB 3
Parts:
- moved J2 82.9 mm to (162.2, 122.8), turned to 90 degrees
- moved J1 64.8 mm to (138.1, 105.0), turned to 180 degrees
- moved J6 49.1 mm to (99.9, 97.4), turned to 0 degrees
- moved J12 47.4 mm to (143.2, 150.8), turned to 0 degrees
- moved J13 44.8 mm to (125.5, 150.8), turned to 0 degrees
- moved D2 42.9 mm to (119.0, 145.7), turned to 90 degrees
- moved R2 42.0 mm to (122.8, 102.5)
- moved D1 39.1 mm to (136.8, 145.7), turned to 90 degrees
- moved U2 39.0 mm to (112.7, 102.5)
- moved J9 37.6 mm to (152.1, 107.6)
- moved R11 26.6 mm to (119.0, 131.8), turned to -90 degrees
- moved R8 24.2 mm to (119.0, 129.2), turned to 90 degrees
- moved R9 20.6 mm to (107.6, 108.9)
- moved R10 19.9 mm to (136.8, 131.8), turned to -90 degrees
- moved U4 19.7 mm to (119.0, 116.5)
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Connections:
- J14 pad 3: /P00 -> /PRES12V1
- J14 pad 4: /P01 -> /PRES12V2
- J15 pad 10: /PRES12V1 -> /P10
- J15 pad 9: /PRES12V2 -> /P11
- U5 pad 1: /P00 -> /P17
- U5 pad 2: /P01 -> /P16
- U5 pad 3: /P02 -> /P15
- U5 pad 4: /P03 -> /P14
- U5 pad 5: /P04 -> /P13
- U5 pad 6: /P05 -> /P12
- U5 pad 7: /P06 -> /P11
- U5 pad 8: /P07 -> /P10
Routing:
- net +5V: track 349.6 -> 76.4 mm, vias 1 -> 0
- net /CMD_PTT: track 92.5 -> 0.00 mm, vias 2 -> 0
- net VCC: track 68.1 -> 0.00 mm
- net /~{INT}: track 85.9 -> 18.8 mm, vias 4 -> 2
- net /SCL: track 95.6 -> 50.4 mm
- net /SDA: track 93.1 -> 50.4 mm
- net /PRES12V1: track 32.9 -> 68.7 mm
- net /P07: track 28.5 -> 0.00 mm
- net /P05: track 28.5 -> 0.00 mm
- net /P00: track 28.5 -> 0.00 mm
- net /P04: track 28.5 -> 0.00 mm
- net /P03: track 28.5 -> 0.00 mm
- net /P02: track 28.5 -> 0.00 mm
- net /P06: track 28.5 -> 0.00 mm
- net /P01: track 28.5 -> 0.00 mm
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Other:
- board size 100.3 x 104.1 mm -> 100.3 x 111.8 mm

Commit message: WIP Update PCB 4
Parts:
- removed U5: ULN2803A, Package_DIP:DIP-18_W7.62mm
- added J11: IN2, Connector_PinHeader_2.54mm:PinHeader_1x02_P2.54mm_Vertical, F.Cu at (107.6, 149.5)
- added J20: OUT1, Connector_PinHeader_2.54mm:PinHeader_1x02_P2.54mm_Vertical, F.Cu at (106.2, 121.6)
- added J21: OUT2, Connector_PinHeader_2.54mm:PinHeader_1x02_P2.54mm_Vertical, F.Cu at (113.8, 121.6)
- added J22: ALIM, Connector_PinHeader_2.54mm:PinHeader_1x02_P2.54mm_Vertical, F.Cu at (101.3, 145.7)
- added J3: IN1, Connector_PinHeader_2.54mm:PinHeader_1x02_P2.54mm_Vertical, F.Cu at (115.2, 149.5)
- moved RLY1 5.02 mm to (146.9, 121.5)
- moved U1 5.02 mm to (141.8, 116.4)
- moved D2 5.02 mm to (124.1, 145.6)
- moved J13 5.02 mm to (130.5, 150.7)
- moved R11 5.02 mm to (124.1, 131.7)
- moved R8 5.02 mm to (124.1, 129.1)
- moved RLY2 5.02 mm to (129.2, 121.5)
- moved D1 5.02 mm to (141.8, 145.6)
- moved J12 5.02 mm to (148.2, 150.7)
- moved R1 5.02 mm to (141.8, 129.1)
- moved R10 5.02 mm to (141.8, 131.7)
- moved R3 5.02 mm to (130.4, 108.8)
- moved R9 5.02 mm to (112.6, 108.8)
- moved U4 5.02 mm to (124.1, 116.4)
- moved J1 1.33 mm to (138.1, 106.3)
Connections:
- J14 pad 3: /PRES12V1 -> /MSG0
- J14 pad 4: /PRES12V2 -> /MSG1
- J14 pad 5: /P02 -> /SEL_CW
- J14 pad 6: /P03 -> /SEL_AM
- J14 pad 7: /P04 -> /CMD_PTT
- J15 pad 10: /P10 -> /CMD_RLY15
- J15 pad 7: /P13 -> /CMD_RLY21
- J15 pad 8: /P12 -> /CMD_RLY25
- J15 pad 9: /P11 -> /CMD_RLY11
- J4 pad 4: /MSG0 -> /PRES12V1
- J4 pad 5: /MSG1 -> /PRES12V2
- J4 pad 6: /SELCW -> /A2
- J4 pad 7: /SELAM -> /A3
- J5 pad 3: /CMD_PTT -> unconnected-(J5-Pin_3-Pad3)
- RLY1 pad 1: /CMD_RLY11 -> /RLY1_1
- RLY1 pad 5: /CMD_RLY15 -> /RLY1_5
- RLY2 pad 1: /CMD_RLY21 -> /RLY2_1
- RLY2 pad 5: /CMD_RLY25 -> /RLY2_5
- U3 pad 13: /SELCW -> /SEL_CW
- U3 pad 5: /SELAM -> /SEL_AM
Routing:
- net +5V: track 76.4 -> 228.2 mm, vias 0 -> 2
- net /CW: track 3.81 -> 113.8 mm, vias 0 -> 2
- net /UTX: track 0.00 -> 85.1 mm, vias 0 -> 2
- net /URX: track 0.00 -> 80.4 mm
- net /DTMF: track 0.00 -> 77.9 mm
- net /~{INT}: track 18.8 -> 92.6 mm, vias 2 -> 4
- net /SDA: track 50.4 -> 120.9 mm, vias 0 -> 1
- net /SCL: track 50.4 -> 117.3 mm, vias 0 -> 1
- net /PRES12V1: track 68.7 -> 3.81 mm
- net /TRX: track 6.91 -> 63.5 mm, vias 0 -> 2
- net /MSG0: track 53.1 -> 0.06 mm
- net /MSG1: track 48.0 -> 0.00 mm
- net /CMD_RLY15: track 43.5 -> 0.00 mm, vias 1 -> 0
- net /MIC: track 2.54 -> 43.5 mm, vias 0 -> 1
- net /PRES12V2: track 44.8 -> 3.81 mm
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